File: kicad/projet_lcd/Ethernet.kicad_sch (KiCad schematic)
At the start: 49 parts, among them U1 LAN8742A-CZ-TR, U3 KMS-1102NL, Y1 25MHz

Commit message: WIP
Other:
- moved on the sheet: R24
Changed lines of the file:
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@@
 	(wire
 		(pts
-			(xy 253 37) (xy 253 32)
+			(xy 250.5 59) (xy 250.5 54)
 		)
 		(stroke
@@
 	(wire
 		(pts
-			(xy 261 32) (xy 261 37)
+			(xy 258.5 54) (xy 258.5 59)
 		)
 		(stroke
@@
 		(lib_name "GND_6")
 		(lib_id "Power:GND")
-		(at 253 37 0)
+		(at 250.5 59 0)
 		(unit 1)
 		(exclude_from_sim no)
@@
 		(fields_autoplaced yes)
 		(property "Reference" "#PWR029"
-			(at 253 43.35 0)
+			(at 250.5 65.35 0)
 			(effects
 				(font
@@
 		)
 		(property "Value" "GND"
-			(at 253 40.81 0)
+			(at 250.5 62.81 0)
 			(effects
 				(font
@@
 		)
 		(property "Footprint" ""
-			(at 253 37 0)
+			(at 250.5 59 0)
 			(effects
 				(font
@@
 		)
 		(property "Datasheet" ""
-			(at 253 37 0)
+			(at 250.5 59 0)
 			(effects
 				(font
@@
 		)
 		(property "Description" "Power symbol creates a global label with name \"GND\" , ground"
-			(at 255.54 47.668 0)
+			(at 253.04 69.668 0)
 			(effects
 				(font
@@
 	(symbol
 		(lib_id "Power:CHASSIS")
-		(at 261 37 0)
+		(at 258.5 59 0)
 		(unit 1)
 		(exclude_from_sim no)
@@
 		(fields_autoplaced yes)
 		(property "Reference" "#PWR030"
-			(at 261 43.35 0)
+			(at 258.5 65.35 0)
 			(effects
 				(font
@@
 		)
 		(property "Value" "CHASSIS"
-			(at 261 40.81 0)
+			(at 258.5 62.81 0)
 			(effects
 				(font
@@
 		)
 		(property "Footprint" ""
-			(at 261 37 0)
+			(at 258.5 59 0)
 			(effects
 				(font
@@
 		)
 		(property "Datasheet" ""
-			(at 261 37 0)
+			(at 258.5 59 0)
 			(effects
 				(font
@@
 		)
 		(property "Description" "Power symbol creates a global label with name \"CHASSIS\" , ground"
-			(at 263.54 47.668 0)
+			(at 261.04 69.668 0)
 			(effects
 				(font
@@
 	(symbol
 		(lib_id "Generiques:R")
-		(at 261 32 90)
+		(at 258.5 54 90)
 		(unit 1)
 		(exclude_from_sim no)
@@
 		(dnp no)
 		(property "Reference" "R24"
-			(at 257 35 90)
+			(at 254.5 57 90)
 			(effects
 				(font
@@
 		)
 		(property "Value" "0"
-			(at 257 30 90)
+			(at 254.5 52 90)
 			(effects
 				(font
@@
 		)
 		(property "Footprint" ""
-			(at 257.254 30.984 90)
+			(at 254.754 52.984 90)
 			(effects
 				(font
@@
 		)
 		(property "Datasheet" "~"
-			(at 257 32 0)
+			(at 254.5 54 0)
 			(effects
 				(font
@@
 		)
 		(property "Description" "Resistor"
-			(at 261 32 0)
+			(at 258.5 54 0)
 			(effects
 				(font
