File: kicad/projet_lcd/Ethernet.kicad_sch (KiCad schematic)
At the start: 48 parts, among them Y3 25MHZ

Commit message: cleanup
Parts:
- removed J3: ~, Connectors:R-RJ45R08P-C000, symbol Connectors:eth_R-RJ45R08P-C000
- added J4: ~, Connectors:R-RJ45R08P-C000, symbol Connectors:R-RJ45R08P-C000
Connections:
- net GND_CHASSIS: now also J4.13 (Shield), J4.14 (Shield)
- net SP1: now also J4.4 (NC), J4.5 (NC)
- net SP2: now also J4.7 (NC), J4.8 (NC)
- net led1: now also J4.9 (LED_Y_A)
- net led2: now also J4.11 (LED_G_A)
- net rx+: now also J4.3 (RX+)
- net rx-: now also J4.6 (RX-)
- net tx+: now also J4.1 (TX+)
- net tx-: now also J4.2 (TX-)
- net at R38.2 (1): now also J4.10 (LED_Y_K)
- net at R40.2 (1): now also J4.12 (LED_G_K)
Changed lines of the file:
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@@
 	)
 	(junction
+		(at 282 121)
+		(diameter 0)
+		(color 0 0 0 0)
+	)
+	(junction
 		(at 56 69)
 		(diameter 0)
@@
 	)
 	(junction
-		(at 258 97)
-		(diameter 0)
-		(color 0 0 0 0)
-	)
-	(junction
 		(at 114 71)
 		(diameter 0)
@@
 	)
 	(junction
-		(at 282 121)
-		(diameter 0)
-		(color 0 0 0 0)
-	)
-	(junction
 		(at 79 44)
 		(diameter 0)
@@
 	)
 	(junction
+		(at 258 97)
+		(diameter 0)
+		(color 0 0 0 0)
+	)
+	(junction
 		(at 27 45)
 		(diameter 0)
@@
 	(wire
 		(pts
-			(xy 282 121) (xy 282 127)
-		)
-		(stroke
-			(width 0)
-			(type default)
-		)
-	)
-	(wire
-		(pts
 			(xy 61 77) (xy 61 109)
 		)
@@
 	(wire
 		(pts
+			(xy 282 118) (xy 282 121)
+		)
+		(stroke
+			(width 0)
+			(type default)
+		)
+	)
+	(wire
+		(pts
 			(xy 224 146) (xy 224 148)
 		)
@@
 	(wire
 		(pts
+			(xy 282 121) (xy 282 127)
+		)
+		(stroke
+			(width 0)
+			(type default)
+		)
+	)
+	(wire
+		(pts
 			(xy 40 109) (xy 61 109)
 		)
@@
 	(wire
 		(pts
-			(xy 282 118) (xy 282 121)
-		)
-		(stroke
-			(width 0)
-			(type default)
-		)
-	)
-	(wire
-		(pts
 			(xy 139 81) (xy 139 85)
 		)
@@
 			)
 		)
-		(property "Description" ""
+		(property "Description" "25Mhz - 8pF - 10ppm"
 			(at 32 145 0)
 			(effects
@@
 	)
 	(symbol
-		(lib_id "Connectors:eth_R-RJ45R08P-C000")
-		(at 258 85 0)
-		(unit 1)
-		(exclude_from_sim no)
-		(in_bom yes)
-		(on_board yes)
-		(dnp no)
-		(fields_autoplaced yes)
-		(property "Reference" "J3"
-			(at 270 81.28 0)
-			(effects
-				(font
-					(size 1.27 1.27)
-				)
-			)
-		)
-		(property "Value" "~"
-			(at 258 85 0)
-			(effects
-				(font
-					(size 1.27 1.27)
-				)
-				(hide yes)
-			)
-		)
-		(property "Footprint" "Connectors:R-RJ45R08P-C000"
-			(at 258 85 0)
-			(effects
-				(font
-					(size 1.27 1.27)
-				)
-				(hide yes)
-			)
-		)
-		(property "Datasheet" "kicad-embed://1912111437_Ckmtw-Shenzhen-Cankemeng-R-RJ45R08P-C000_C386757.pdf"
-			(at 271 130 0)
-			(effects
-				(font
-					(size 1.27 1.27)
-				)
-				(hide yes)
-			)
-		)
-		(property "Description" "RJ45 Receptacle / Shielded / Bend insert / With LED"
-			(at 270 127 0)
-			(effects
-				(font
-					(size 1.27 1.27)
-				)
-				(hide yes)
-			)
-		)
-		(property "Part #" "R-RJ45R08P-C000"
-			(at 269 133 0)
-			(effects
-				(font
-					(size 1.27 1.27)
-				)
-				(hide yes)
-			)
-		)
-		(property "LCSC Part #" "C386757"
-			(at 269 136 0)
-			(effects
-				(font
-					(size 1.27 1.27)
-				)
-				(hide yes)
-			)
-		)
-		(pin "8"
-		)
-		(pin "6"
-		)
-		(pin "10"
-		)
-		(pin "5"
-		)
-		(pin "3"
-		)
-		(pin "13"
-		)
-		(pin "14"
-		)
-		(pin "12"
-		)
-		(pin "11"
-		)
-		(pin "4"
-		)
-		(pin "1"
-		)
-		(pin "7"
-		)
-		(pin "2"
-		)
-		(pin "9"
-		)
-		(instances
-			(project ""
-				(path "/b3ce22de-813e-4a84-80c2-bec39c904000/4f5f892b-036b-4e71-84df-7e1dbf92e07c"
-					(reference "J3")
-					(unit 1)
-				)
-			)
-		)
-	)
-	(symbol
 		(lib_id "Generics:C")
 		(at 51 152 90)
@@
 					(unit 1)
 				)
+			)
+		)
+	)
+	(symbol
+		(lib_id "Connectors:R-RJ45R08P-C000")
+		(at 258 85 0)
+		(unit 1)
+		(exclude_from_sim no)
+		(in_bom yes)
+		(on_board yes)
+		(dnp no)
+		(fields_autoplaced yes)
+		(property "Reference" "J4"
+			(at 270 80.48 0)
+			(effects
+				(font
+					(size 1.27 1.27)
+				)
+			)
+		)
+		(property "Value" "~"
+			(at 258 85 0)
+			(effects
+				(font
+					(size 1.27 1.27)
+				)
+				(hide yes)
+			)
+		)
+		(property "Footprint" "Connectors:R-RJ45R08P-C000"
+			(at 258 85 0)
+			(effects
+				(font
+					(size 1.27 1.27)
+				)
+				(hide yes)
+			)
+		)
+		(property "Datasheet" "kicad-embed://1912111437_Ckmtw-Shenzhen-Cankemeng-R-RJ45R08P-C000_C386757.pdf"
+			(at 271 130 0)
+			(effects
+				(font
+					(size 1.27 1.27)
+				)
+				(hide yes)
+			)
+		)
+		(property "Description" "RJ45 Receptacle / Shielded / Bend insert / With LED"
+			(at 270 127 0)
+			(effects
+				(font
+					(size 1.27 1.27)
+				)
+				(hide yes)
+			)
+		)
+		(property "Part#" "R-RJ45R08P-C000"
+			(at 269 133 0)
+			(effects
+				(font
+					(size 1.27 1.27)
+				)
+				(hide yes)
+			)
+		)
+		(property "LCSC Part#" "C386757"
+			(at 269 136 0)
+			(effects
+				(font
+					(size 1.27 1.27)
+				)
+				(hide yes)
+			)
+		)
+		(pin "7"
+		)
+		(pin "14"
+		)
+		(pin "6"
+		)
+		(pin "8"
+		)
+		(pin "2"
+		)
+		(pin "12"
+		)
+		(pin "1"
+		)
+		(pin "3"
+		)
+		(pin "4"
+		)
+		(pin "5"
+		)
+		(pin "11"
+		)
+		(pin "10"
+		)
+		(pin "9"
+		)
+		(pin "13"
+		)
+		(instances
+			(project ""
+				(path "/b3ce22de-813e-4a84-80c2-bec39c904000/4f5f892b-036b-4e71-84df-7e1dbf92e07c"
+					(reference "J4")
+					(unit 1)
+				)

Commit message: DRC / ERC ok
Other:
- note added: "Paires differentielles !!!"
Changed lines of the file:
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@@
+		)
+	)
+	(text "Paires differentielles !!!"
+		(exclude_from_sim no)
+		(at 152 112 0)
+		(effects
+			(font
+				(size 1.27 1.27)
+				(color 255 0 0 1)
+			)
 		)
 	)
@@
 		)
 	)
-	(text_box "WTF ???"
-		(exclude_from_sim no)
-		(at 14 130 0)
-		(size 10 3)
-		(margins 0.9525 0.9525 0.9525 0.9525)
-		(stroke
-			(width 0)
-			(type solid)
-		)
-		(fill
-			(type none)
-		)
-		(effects
-			(font
-				(size 1.27 1.27)
-				(color 255 0 0 1)
-			)
-			(justify left top)
-		)
-	)
