File: kicad/projet_lcd/projet_lcd.kicad_sch (KiCad schematic)
At the start: 49 parts, among them U1 KMS-1102NL, U2 LAN8742A-CZ-TR, Y1 25MHz

Commit message: Work in progress
Parts:
- removed C1, C2, C3, C4: 22pF, symbol Generiques:C
- removed C10, C11, C12: 10nF, symbol Generiques:C
- removed C13, C18: 10uF, symbol Generiques:C_Polarized
- removed C14: 470pF, symbol Generiques:C_Polarized
- removed C15: 1uF, symbol Generiques:C_Polarized
- removed C16, C17: 30pF, symbol Generiques:C
- removed C19: 100nF, symbol Generiques:C
- removed C5: 22nF, symbol Generiques:C_Polarized
- removed C6, C7: 1nF, symbol Generiques:C
- removed C8, C9: TBD, symbol Generiques:C
- removed CN1: ~, symbol Connectors:RJ45_with_Leds
- removed FB1: FerriteBead, symbol Generiques:FerriteBead
- removed R1, R2, R3, R4: 49R9, symbol Generiques:R
- removed R10: 12.1K, symbol Generiques:R
- removed R11, R12, R13: 10, symbol Generiques:R
- removed R14, R15, R17, R18, R19, R23: 10K, symbol Generiques:R
- removed R16: 1.5K, symbol Generiques:R
- removed R20, R21: 270R, symbol Generiques:R
- removed R22, R24: 0, symbol Generiques:R
- removed R5, R6, R7, R8: 75R, symbol Generiques:R
- removed R9: 33, symbol Generiques:R
- removed U1: KMS-1102NL, symbol Divers:KMS-1102NL
- removed U2: LAN8742A-CZ-TR, symbol Chips:LAN8742A
- removed U3: ~, symbol Diodes:USBLC6-4
- removed Y1: 25MHz, symbol Generiques:Crystal
Other:
- added sheet Ethernet (Main.kicad_sch)
- added sheet POE (POE.kicad_sch)
- note removed: "An additional external 1.0M resistor across the crystal is not required. The necessary resistance has been designed into the LAN8742 internally."
- note removed: "Bulk capacitors for the ferrite bead"
- note removed: "Cmagterm"
- note removed: "Crjterm"
- note removed: "Découplage de VDD1A et VDD2A 0603 or smaller"
- note removed: "Découplage de VDDIO 0603 or smaller"
- note removed: "Paires differentielles 100 Ohms !!!"

Commit message: wip
Parts:
- added U7: ~, symbol Ethernet:LAN8742A
Other:
- added sheet stm32 (stm32.kicad_sch)
- sheet Ethernet: file Main.kicad_sch -> Ethernet.kicad_sch
- sheet Ethernet ports: added CT1, CT2, SP1, SP2; removed none
- sheet POE ports: added CT1, CT2, SP1, SP2; removed none

Commit message: WIP
Parts:
- removed U7: ~, symbol Ethernet:LAN8742A
Other:
- sheet stm32 ports: added RMII_CRS_DV, RMII_MDC, RMII_MDIO, RMII_REFCLK, RMII_RXD0, RMII_RXD1, RMII_TXD0, RMII_TXD1, RMII_TXEN, UDB_DM, UDB_DP, ~{RST}; removed none
Changed lines of the file:
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@@
+	(wire
+		(pts
+			(xy 108 56) (xy 160 56)
+		)
+		(stroke
+			(width 0)
+			(type default)
+		)
+	)
+	(wire
+		(pts
+			(xy 108 44) (xy 160 44)
+		)
+		(stroke
+			(width 0)
+			(type default)
+		)
+	)
+	(wire
+		(pts
+			(xy 108 38) (xy 160 38)
+		)
+		(stroke
+			(width 0)
+			(type default)
+		)
+	)
+	(wire
+		(pts
+			(xy 108 47) (xy 160 47)
+		)
+		(stroke
+			(width 0)
+			(type default)
+		)
+	)
+	(wire
+		(pts
+			(xy 108 50) (xy 160 50)
+		)
+		(stroke
+			(width 0)
+			(type default)
+		)
+	)
 	(wire
 		(pts
@@
 	(wire
 		(pts
+			(xy 108 41) (xy 160 41)
+		)
+		(stroke
+			(width 0)
+			(type default)
+		)
+	)
+	(wire
+		(pts
 			(xy 185 61) (xy 185 75)
 		)
@@
 		)
 	)
-	(symbol
-		(lib_id "Ethernet:LAN8742A")
-		(at 53 115 0)
-		(unit 1)
-		(exclude_from_sim no)
-		(in_bom yes)
-		(on_board yes)
-		(dnp no)
-		(fields_autoplaced yes)
-		(property "Reference" "U7"
-			(at 56 108 0)
-			(do_not_autoplace yes)
-			(effects
-				(font
-					(size 1.25 1.25)
-				)
-				(justify left)
-			)
-		)
-		(property "Value" "~"
-			(at 64.5 170.5 0)
-			(do_not_autoplace yes)
-			(effects
-				(font
-					(size 1.25 1.25)
-				)
-				(hide yes)
-			)
-		)
-		(property "Footprint" ""
-			(at 53 176 0)
-			(effects
-				(font
-					(size 1.25 1.25)
-				)
-				(hide yes)
-			)
-		)
-		(property "Datasheet" ""
-			(at 53 176 0)
-			(effects
-				(font
-					(size 1.25 1.25)
-				)
-				(hide yes)
-			)
-		)
-		(property "Description" "Ethernet Controller"
-			(at 76.5 181 0)
-			(effects
-				(font
-					(size 1.25 1.25)
-				)
-				(hide yes)
-			)
-		)
-		(property "Part#" "LAN8742A-CZ-TR"
-			(at 56 170.5 0)
-			(do_not_autoplace yes)
-			(effects
-				(font
-					(size 1.25 1.25)
-				)
-				(justify left)
-			)
-		)
-		(property "Comments" ""
-			(at 53 115 0)
-			(effects
-				(font
-					(size 1.25 1.25)
-				)
-				(hide yes)
-			)
-		)
-		(pin "13"
-		)
-		(pin "12"
-		)
-		(pin "10"
-		)
-		(pin "21"
-		)
-		(pin "5"
-		)
-		(pin "7"
-		)
-		(pin "24"
-		)
-		(pin "20"
-		)
-		(pin "15"
-		)
-		(pin "18"
-		)
-		(pin "1"
-		)
-		(pin "6"
-		)
-		(pin "17"
-		)
-		(pin "3"
-			(alternate "LED1")
-		)
-		(pin "4"
-		)
-		(pin "23"
-		)
-		(pin "22"
-		)
-		(pin "25"
-		)
-		(pin "11"
-		)
-		(pin "14"
-		)
-		(pin "9"
-		)
-		(pin "19"
-		)
-		(pin "16"
-		)
-		(pin "8"
-		)
-		(pin "2"
-		)
-		(instances
-			(project ""
-				(path "/b3ce22de-813e-4a84-80c2-bec39c904000"
-					(reference "U7")
-					(unit 1)
-				)
-			)
+	(wire
+		(pts
+			(xy 108 32) (xy 160 32)
+		)
+		(stroke
+			(width 0)
+			(type default)
+		)
+	)
+	(wire
+		(pts
+			(xy 108 59) (xy 160 59)
+		)
+		(stroke
+			(width 0)
+			(type default)
+		)
+	)
+	(wire
+		(pts
+			(xy 108 53) (xy 160 53)
+		)
+		(stroke
+			(width 0)
+			(type default)
+		)
+	)
+	(wire
+		(pts
+			(xy 108 35) (xy 160 35)
+		)
+		(stroke
+			(width 0)
+			(type default)
 		)
 	)
@@
 			)
 		)
+		(pin "UDB_DP" bidirectional
+			(at 79.5 74 270)
+			(effects
+				(font
+					(size 1.27 1.27)
+				)
+				(justify left)
+			)
+		)
+		(pin "~{RST}" input
+			(at 108 59 0)
+			(effects
+				(font
+					(size 1.27 1.27)
+				)
+				(justify right)
+			)
+		)
+		(pin "RMII_TXD0" output
+			(at 108 32 0)
+			(effects
+				(font
+					(size 1.27 1.27)
+				)
+				(justify right)
+			)
+		)
+		(pin "RMII_TXD1" output
+			(at 108 35 0)
+			(effects
+				(font
+					(size 1.27 1.27)
+				)
+				(justify right)
+			)
+		)
+		(pin "RMII_REFCLK" input
+			(at 108 56 0)
+			(effects
+				(font
+					(size 1.27 1.27)
+				)
+				(justify right)
+			)
+		)
+		(pin "RMII_TXEN" output
+			(at 108 38 0)
+			(effects
+				(font
+					(size 1.27 1.27)
+				)
+				(justify right)
+			)
+		)
+		(pin "RMII_MDIO" bidirectional
+			(at 108 50 0)
+			(effects
+				(font
+					(size 1.27 1.27)
+				)
+				(justify right)
+			)
+		)
+		(pin "RMII_CRS_DV" input
+			(at 108 47 0)
+			(effects
+				(font
+					(size 1.27 1.27)
+				)
+				(justify right)
+			)
+		)
+		(pin "UDB_DM" bidirectional
+			(at 82.5 74 270)
+			(effects
+				(font
+					(size 1.27 1.27)
+				)
+				(justify left)
+			)
+		)
+		(pin "RMII_MDC" output
+			(at 108 53 0)
+			(effects
+				(font
+					(size 1.27 1.27)
+				)
+				(justify right)
+			)
+		)
+		(pin "RMII_RXD0" input
+			(at 108 41 0)
+			(effects
+				(font
+					(size 1.27 1.27)
+				)
+				(justify right)
+			)
+		)
+		(pin "RMII_RXD1" input
+			(at 108 44 0)
+			(effects
+				(font
+					(size 1.27 1.27)
+				)
+				(justify right)
+			)
+		)
