File: kicad/projet_lcd/stm32.kicad_sch (KiCad schematic)
At the start: 0 parts

Commit message: WIP
Parts:
- added C41, C42, C43, C44, C45, C47, C48, C49: 100nF, symbol Generics:C
- added C46: 4.7uF, symbol Generics:C_Polarized
- added C50: 1uF, symbol Generics:C_Polarized
- added C51, C54, C55, C56, C57: NI, symbol Generics:C
- added C52, C53: 2.2uF, symbol Generics:C
- added C58: 0.1uF, symbol Generics:C
- added J1: ~, symbol PCB_Utils:J_SWD
- added R42: NI, symbol Generics:R
- added SW_RESET: ~, symbol Generics:SW_PushButton
- added U7: ~, Microcontrollers:STM32H563VIT6, symbol MicroControllers:STM32H563VIT6
- added Y2: NI, symbol Generics:Y
- added Y3: 32.768KHz, symbol Generics:Y
Connections:
- new net: C57.2, U7.9 (PC15-OSC32_OUT), Y3.2
- new net: C54.2, U7.12 (PH0-OSC_IN), Y2.1
- new net: C55.2, U7.13 (PH1-OSC_OUT), Y2.2
- new net: C51.2, R42.2 (1), U7.21 (VREF+)
- new net: C52.2, C53.2, U7.48 (VCAP), U7.98 (VCAP)
- new net: C56.2, U7.8 (PC14-OSC32_IN), Y3.1
- new net +3.3V: C41.2, C42.2, C43.2, C44.2, C45.2, C46.P, C47.2, C48.2, C49.2, C50.P, J1.1 (VDD), R42.1, U7.100 (VDD), U7.11 (VDD), U7.22 (VDDA), U7.28 (VDD), U7.50 (VDD), U7.6 (VBAT), U7.73 (VDDUSB), U7.75 (VDD)
- new net GND: C41.1, C42.1, C43.1, C44.1, C45.1, C46.N, C47.1, C48.1, C49.1, C50.N, C51.1, C52.1, C53.1, C54.1, C55.1, C56.1, C57.1, C58.1, J1.3 (GND), SW_RESET.2, U7.10 (VSS), U7.19 (VSSA), U7.20 (VREF-), U7.27 (VSS), U7.49 (VSS), U7.74 (VSS), U7.94 (BOOT0), U7.99 (VSS)
- new net RMII_CRS_DV: U7.32 (PA7)
- new net RMII_MDC: U7.16 (PC1)
- new net RMII_MDIO: U7.25 (PA2)
- new net RMII_REFCLK: U7.24 (PA1)
- new net RMII_RXD0: U7.33 (PC4)
- new net RMII_RXD1: U7.34 (PC5)
- new net RMII_TXD0: U7.51 (PB12)
- new net RMII_TXD1: U7.54 (PB15)
- new net RMII_TXEN: U7.30 (PA5)
- new net SWCLK: J1.2 (SWCLK), U7.76 (PA14)
- new net SWD_RST: C58.2, J1.5 (NRST), SW_RESET.1, U7.14 (NRST)
- new net SWIO: J1.4 (SWDIO), U7.72 (PA13)
- new net SWO: J1.6 (SWO), U7.89 (PB3)
- new net UDB_DM: U7.70 (PA11)
- new net UDB_DP: U7.71 (PA12)
- new net ~{RST}: U7.36 (PB1)
Other:
- note added: "4 to 50 MHz"
- note added: "ESR Max 100mΩ"
- note added: "PCB and MCU pin capacitance must be included (10 pF can be used as a rough estimate of the combined pin and board capacitance) when sizing CL1 and CL2."
- note added: "SOLDER BRIDGE ?"
- note added: "TODO: ECRAN USB USART SORTIE DES PORTS INUTILISES SUR HEADER"
