File: kicad/projet_lcd/POE.kicad_sch (KiCad schematic)
At the start: 64 parts, among them Q1 FOD817A3SD, T1 749119950

Commit message: EOD
Parts:
- removed C35: 1.5nF, Generics:C_0603, symbol Generics:C
- removed DB1, DB2: ~, symbol Generics:DB
- removed R16: 0R, Generics:R_0603, symbol Generics:R
- removed T1: 749119950, symbol Inductors:749119950
- added C20: 1nF, Generics:C_1808, symbol Generics:C
- added C32, C33, C34, C41, C42, C43, C44: 1nF, Generics:C_0603, symbol Generics:C
- added C37: 1uF, Generics:C_1210, symbol Generics:C
- added C45: 1.5nF, Generics:C_0805, symbol Generics:C
- added D10, D11, D12, D13, D4, D5, D6, D7: ~, Generics:SMA, symbol Generics:D
- added D8: ~, Generics:SMA, symbol Generics:D_TVS
- added R18: 0R, Generics:R_0805, symbol Generics:R
- added T1: ~, Ethernet:749119950, symbol Ethernet:749119950
- C21: renamed from C20; footprint (none) -> Generics:C_0805; LCSC Part # (none) -> C107135
- C22: renamed from C19; footprint (none) -> Generics:C_0805; LCSC Part # (none) -> C1717
- C23: renamed from C21; footprint (none) -> Generics:C_0603; LCSC Part # (none) -> C15849
- C24: renamed from C22; footprint (none) -> Generics:C_1210; LCSC Part # (none) -> C7432783
- C25: renamed from C23; LCSC Part # (none) -> C2983415
- C26: renamed from C24; footprint (none) -> Generics:C_1210; now left out of the parts list
- C27: renamed from C25; footprint (none) -> Generics:C_1210
- C28: renamed from C26; footprint (none) -> Generics:C_1210
- C29: renamed from C27; footprint (none) -> Generics:C_0805; LCSC Part # (none) -> C7500383
- C30: renamed from C28; footprint (none) -> Generics:C_0805; LCSC Part # (none) -> C28323
- C31: value 1uF -> 1nF; footprint (none) -> Generics:C_0603; Comments 100V -> 1nF / 100V / X7R; now not fitted; now left out of the parts list
- C35: renamed from C29; LCSC Part # (none) -> C487173
- C36: renamed from C30; footprint (none) -> Generics:C_1210; LCSC Part # (none) -> C91151
- C38: renamed from C32; footprint (none) -> Generics:C_0603; LCSC Part # (none) -> C43253
- C39: renamed from C34; footprint (none) -> Generics:C_0805; LCSC Part # (none) -> C28233
- C40: renamed from C41; footprint Generics:C_0603 -> Generics:C_0805; LCSC Part # C14663 -> C49678
- C46: renamed from C36; footprint Generics:C_0603 -> Generics:C_0805
- C47: renamed from C37; footprint Generics:C_0603 -> Generics:C_1808; Comments (none) -> 3000V; LCSC Part # C1588 -> C173224
- D1: LCSC Part # (none) -> C5746878; Part# NI -> (none)
- D2: footprint (none) -> Generics:SMA; LCSC Part # (none) -> C437609
- D3: footprint (none) -> Generics:SOD-123; LCSC Part # (none) -> C81598
- D9: renamed from D4; footprint Generics:D_LED_0603 -> Generics:D_LED_0805; LCSC Part # (none) -> C84256
- FB1, FB2: footprint (none) -> Generics:L_0805; Comments (none) -> 150mΩ ±25% 600Ω@100MHz 0805 Ferrite Beads ROHS; LCSC Part # (none) -> C2661857; Part# (none) -> 742792040
- L1: value NI -> 0.16uH; LCSC Part # (none) -> C18236235
- Q1: LCSC Part # (none) -> C128788
- R10: renamed from R7; footprint (none) -> Generics:R_0805; Part# (none) -> C17850
- R11: renamed from R9; footprint Generics:R_0402 -> Generics:R_0805; LCSC Part # C25077 -> C17415
- R12: renamed from R10; footprint Generics:R_0402 -> Generics:R_0805; LCSC Part # C25900 -> C17673
- R13: renamed from R11; footprint Generics:R_0402 -> Generics:R_0805; LCSC Part # C137936 -> C17818
- R14: renamed from R12; footprint Generics:R_0402 -> Generics:R_0805; LCSC Part # C15011 -> C35928
- R15: footprint Generics:R_0603 -> Generics:R_0805; LCSC Part # (none) -> C17513
- R16: renamed from R13; footprint (none) -> Generics:R_0805; LCSC Part # (none) -> C2930222
- R17: renamed from R14; footprint Generics:R_0603 -> Generics:R_0805; now left out of the parts list
- R19: renamed from R17; footprint (none) -> Generics:R_0805; LCSC Part # (none) -> C384088
- R20: renamed from R18; footprint Generics:R_0402 -> Generics:R_0805; LCSC Part # C132157 -> C2933295
- R4: renamed from R2; footprint (none) -> Generics:R_0805; LCSC Part # (none) -> C844811
- R5: renamed from R4; footprint (none) -> Generics:R_0805; LCSC Part # (none) -> C17840
- R6: renamed from R3; footprint (none) -> Generics:R_0805; LCSC Part # (none) -> C144544
- R7: renamed from R5; footprint (none) -> Generics:R_0805; LCSC Part # (none) -> C17477
- R8: footprint (none) -> Generics:R_0805; LCSC Part # (none) -> C17660
- R9: renamed from R6; footprint (none) -> Generics:R_0805; LCSC Part # (none) -> C101593
- U2: footprint (none) -> Ethernet:SI3404-A-GMR
- U3: LCSC Part # (none) -> C2156583; PART# TL431 -> (none); Part# (none) -> TL431
- U4: footprint (none) -> Voltage_Regulators:AMS1117-3.3; LCSC Part # (none) -> C6186
- renumbered C38 to C48, C39 to C49, TP9 to TP10, TP10 to TP11, TP11 to TP2, TP2 to TP3, TP3 to TP4, TP4 to TP5, TP5 to TP6, TP6 to TP7, TP7 to TP8, TP8 to TP9
Connections:
- net +3.3V: now also U4.2 (Vout), U4.4 (Tab); no longer U4.Vout
- net +5V: now also U4.3 (Vin), C20.2; no longer U4.Vin
- net CT1: now also C31.1, C41.2, D10.K, D4.A
- net CT2: now also C32.1, C42.2, D11.K, D5.A
- net GND: now also T1.10, T1.9
- net SP1: now also C33.1, C43.2, D12.K, D6.A
- net SP2: now also C34.1, C44.2, D13.K, D7.A
- net vpos: now also C20.1, C37.2, T1.4; no longer C31.2
- net vss: now also C37.1, T1.1; no longer C31.1
- net at R7.2 (1): now also T1.2
- net at D2.A, TP5.1, U2.18 (SWO): now also T1.3
- net at C22.2, D1.A: now also T1.7, T1.8
- net at Q1.K, U3.K: now also C45.2
- net at FB1.1: now also C31.2, C32.2, C33.2, C34.2, D4.K, D5.K, D6.K, D7.K, D8.K
- net at R14.1, R20.1, U3.Ref: now also R18.2 (1)
- net at FB2.1: now also C41.1, C42.1, C43.1, C44.1, D10.A, D11.A, D12.A, D13.A, D8.A
- new net: C45.1, R18.1
Other:
- note added: "POE Power Supply"
- note removed: "S1B"
- moved on the sheet: C21, C30, C35, C36, C38, C39, C49, FB1, R5, R8, TP1, TP10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

Commit message: EOD \o/
Parts:
- removed C25: 560uF, symbol Generics:C_Polarized
- removed C35: 12uF, symbol Generics:C_Polarized
- removed D9: ~, Generics:D_LED_0805, symbol Generics:D_LED
- removed Q1: FOD817A3SD, symbol Generics:OP
- removed TP11: ~, PCB_Utils:TP_1.5, symbol PCB_Utils:TP
- added C32: 560uF, Passives:CAP-SMD_BD10.0-L10.3-W10.3-LS11.0-FD-1, symbol Passives:C_SMD_ALU_560uF_6V3
- added C42: 12uF, symbol Generics:C_alt
- added D9: ~, Generics:D_LED_0603, symbol Generics:D_LED_red
- added Q1: FOD817A3SD, Optoelectronics:FOD817A3SD, symbol Optoelectronics:OPTO_FOD817A3SD
- L1: value 0.16uH -> 160nH; footprint (none) -> Passives:IND-SMD_L5.5-W5.3; symbol Generics:L -> Passives:L_160nH_SMD; Manufacturer (none) -> YJYCOIN; Part# (none) -> YSPIT0530A-R16M
- R15: value 1K -> 150R; footprint Generics:R_0805 -> Generics:R_0603; LCSC Part # C17513 -> C22808
- U3: footprint (none) -> Voltage_Regulators:TL431
- renumbered C20 to C27, C21 to C28, C22 to C29, C23 to C30, C24 to C31, C26 to C33, C27 to C34, C28 to C35, C29 to C36, C30 to C37, C31 to C38, C32 to C39, C33 to C40, C34 to C41, C36 to C43, C37 to C44, C38 to C45, C39 to C46, C40 to C47, C41 to C48, C42 to C49, C43 to C50, C44 to C51, C45 to C52, C46 to C53, C47 to C54, C48 to C55, C49 to C56, TP9 to TP10, TP10 to TP11, TP12 to TP13, TP1 to TP2, TP2 to TP3, TP3 to TP4, TP4 to TP5, TP5 to TP6, TP6 to TP7, TP7 to TP8, TP8 to TP9
Connections:
- net +5V: now also C32.P
- net GND: now also C32.N, D9.K
- net vpos: now also C42.2
- net at C52.2, U3.K: now also Q1.K
- net at R15.1: now also D9.A
- net at R13.1: now also Q1.A
- net at R12.1, R17.2 (1), TP10.1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: now also Q1.C
- net vss renamed VSS
- net VSS: now also C42.1, Q1.E
Other:
- moved on the sheet: C47, C54, R7
