File: kicad/projet_lcd/USB.kicad_sch (KiCad schematic)
At the start: 7 parts

Commit message: EOD \o/
Parts:
- renumbered J8 to J4, R50 to R45, R45 to R46, R46 to R47, R47 to R48, R48 to R49, R49 to R50
Changed lines of the file:
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@@
 		(dnp no)
 		(fields_autoplaced yes)
-		(property "Reference" "#PWR076"
+		(property "Reference" "#PWR081"
 			(at 133 115.35 0)
 			(effects
@@
 			(project ""
 				(path "/b3ce22de-813e-4a84-80c2-bec39c904000/c6fab658-f544-4247-906b-fdb14f28513d"
-					(reference "#PWR076")
+					(reference "#PWR081")
 					(unit 1)
 				)
@@
 		(dnp no)
 		(fields_autoplaced yes)
-		(property "Reference" "R47"
+		(property "Reference" "R48"
 			(at 108 89 0)
 			(do_not_autoplace yes)
@@
 			(project "projet_lcd"
 				(path "/b3ce22de-813e-4a84-80c2-bec39c904000/c6fab658-f544-4247-906b-fdb14f28513d"
-					(reference "R47")
+					(reference "R48")
 					(unit 1)
 				)
@@
 		(dnp no)
 		(fields_autoplaced yes)
-		(property "Reference" "R50"
+		(property "Reference" "R45"
 			(at 160 89 0)
 			(do_not_autoplace yes)
@@
 			(project "projet_lcd"
 				(path "/b3ce22de-813e-4a84-80c2-bec39c904000/c6fab658-f544-4247-906b-fdb14f28513d"
-					(reference "R50")
+					(reference "R45")
 					(unit 1)
 				)
@@
 		(dnp no)
 		(fields_autoplaced yes)
-		(property "Reference" "#PWR075"
+		(property "Reference" "#PWR082"
 			(at 155 116.35 0)
 			(effects
@@
 			(project ""
 				(path "/b3ce22de-813e-4a84-80c2-bec39c904000/c6fab658-f544-4247-906b-fdb14f28513d"
-					(reference "#PWR075")
+					(reference "#PWR082")
 					(unit 1)
 				)
@@
 		(dnp no)
 		(fields_autoplaced yes)
-		(property "Reference" "R48"
+		(property "Reference" "R49"
 			(at 116 89 0)
 			(do_not_autoplace yes)
@@
 			(project "projet_lcd"
 				(path "/b3ce22de-813e-4a84-80c2-bec39c904000/c6fab658-f544-4247-906b-fdb14f28513d"
-					(reference "R48")
+					(reference "R49")
 					(unit 1)
 				)
@@
 		(on_board yes)
 		(dnp no)
-		(property "Reference" "#PWR077"
+		(property "Reference" "#PWR080"
 			(at 149 103 0)
 			(effects
@@
 			(project ""
 				(path "/b3ce22de-813e-4a84-80c2-bec39c904000/c6fab658-f544-4247-906b-fdb14f28513d"
-					(reference "#PWR077")
+					(reference "#PWR080")
 					(unit 1)
 				)
@@
 		(on_board yes)
 		(dnp no)
-		(property "Reference" "J8"
+		(property "Reference" "J4"
 			(at 146 91 0)
 			(effects
@@
 			(project ""
 				(path "/b3ce22de-813e-4a84-80c2-bec39c904000/c6fab658-f544-4247-906b-fdb14f28513d"
-					(reference "J8")
+					(reference "J4")
 					(unit 1)
 				)
@@
 		(dnp no)
 		(fields_autoplaced yes)
-		(property "Reference" "#PWR074"
+		(property "Reference" "#PWR079"
 			(at 94 93 0)
 			(effects
@@
 			(project ""
 				(path "/b3ce22de-813e-4a84-80c2-bec39c904000/c6fab658-f544-4247-906b-fdb14f28513d"
-					(reference "#PWR074")
+					(reference "#PWR079")
 					(unit 1)
 				)
@@
 		(dnp no)
 		(fields_autoplaced yes)
-		(property "Reference" "R49"
+		(property "Reference" "R50"
 			(at 125 89 0)
 			(do_not_autoplace yes)
@@
 			(project "projet_lcd"
 				(path "/b3ce22de-813e-4a84-80c2-bec39c904000/c6fab658-f544-4247-906b-fdb14f28513d"
-					(reference "R49")
+					(reference "R50")
 					(unit 1)
 				)
@@
 		(dnp no)
 		(fields_autoplaced yes)
-		(property "Reference" "R46"
+		(property "Reference" "R47"
 			(at 100 89 0)
 			(do_not_autoplace yes)
@@
 			(project "projet_lcd"
 				(path "/b3ce22de-813e-4a84-80c2-bec39c904000/c6fab658-f544-4247-906b-fdb14f28513d"
-					(reference "R46")
+					(reference "R47")
 					(unit 1)
 				)
@@
 		(dnp no)
 		(fields_autoplaced yes)
-		(property "Reference" "R45"
+		(property "Reference" "R46"
 			(at 92 89 0)
 			(do_not_autoplace yes)
@@
 			(project ""
 				(path "/b3ce22de-813e-4a84-80c2-bec39c904000/c6fab658-f544-4247-906b-fdb14f28513d"
-					(reference "R45")
-					(unit 1)
-				)
+					(reference "R46")
+					(unit 1)
+				)
