File: kicad/projet_lcd/io_connectors.kicad_sch (KiCad schematic)
At the start: 2 parts

Commit message: on avance !
Parts:
- added J3: ~, Connectors:FH34SRJ-18S-0.5SH(50), symbol Connectors:FH34SRJ-18S-0.5SH(50)
- added J8: ~, Generics:Header_1x12_2.54_TH_labels, symbol Generics:J_Connector_1x12
- added Q2: AO3400A, Transistors:SOT-23-3_L2.9-W1.3-P1.90-LS2.4-BR, symbol Transistors:AO3400A
- added R52, R55, R56, R57: 33, symbol Generics:R
- added R53: 10k, Generics:R_0603, symbol Generics:R
- added R54: 33R, Generics:R_0402, symbol Generics:R
- added TP14, TP15, TP16, TP17: ~, PCB_Utils:TP_1.5, symbol PCB_Utils:TP
Connections:
- net +3.3V: now also J3.10; no longer J5.1, J6.1
- net GND: now also J3.11, J3.12, J3.18, J3.19, J3.20, J8.12, Q2.2 (S), R53.1
- new net: J3.1, TP14.1
- new net: J3.2, TP15.1
- new net: J3.3, TP16.1
- new net: J3.4, TP17.1
- new net: J3.5, R57.2 (1)
- new net: J3.6, R56.2 (1)
- new net: J3.7, R52.2 (1)
- new net: J3.8, R55.2 (1)
- new net: Q2.3 (D), R52.1, R55.1, R56.1, R57.1
- new net: Q2.1 (G), R53.2 (1), R54.1
- new net +5V: J3.9
- new net DISPLAY_CS: J3.14
- new net DISPLAY_PWM: R54.2 (1)
- new net DISPLAY_RS: J3.15
- new net DISPLAY_RST: J3.17
- new net DISPLAY_SCL: J3.16
- new net DISPLAY_SDA: J3.13
- new net OUTPUT_0: J8.2
- new net OUTPUT_1: J8.3
- new net OUTPUT_2: J8.4
- new net OUTPUT_3: J8.5
- new net OUTPUT_4: J8.6
- new net OUTPUT_5: J8.7
- new net OUTPUT_6: J8.8
- new net OUTPUT_7: J8.9
- new net OUTPUT_8: J8.10
- new net OUTPUT_9: J8.11
- new net Vaux_3V3: J5.1, J6.1, J8.1
Other:
- moved on the sheet: J5, J6

Commit message: routage en cours
Parts:
- J5: PIN_01 VCC -> ## PIN1; PIN_02 SDA -> ## PIN2; PIN_03 SCL -> ## PIN3; PIN_04 GND -> ## PIN4
- R52, R55, R56, R57: footprint (none) -> Generics:R_0805
Other:
- moved on the sheet: J8
Changed lines of the file:
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@@
 	(wire
 		(pts
-			(xy 242 117) (xy 250 117)
-		)
-		(stroke
-			(width 0)
-			(type default)
-		)
-	)
-	(wire
-		(pts
-			(xy 247 108) (xy 250 108)
+			(xy 203 118) (xy 211 118)
+		)
+		(stroke
+			(width 0)
+			(type default)
+		)
+	)
+	(wire
+		(pts
+			(xy 208 109) (xy 211 109)
 		)
 		(stroke
@@
 	(wire
 		(pts
-			(xy 242 111) (xy 250 111)
+			(xy 203 112) (xy 211 112)
 		)
 		(stroke
@@
 	(wire
 		(pts
-			(xy 242 132) (xy 250 132)
+			(xy 203 133) (xy 211 133)
 		)
 		(stroke
@@
 	(wire
 		(pts
-			(xy 242 135) (xy 250 135)
+			(xy 203 136) (xy 211 136)
 		)
 		(stroke
@@
 	(wire
 		(pts
-			(xy 242 120) (xy 250 120)
+			(xy 203 121) (xy 211 121)
 		)
 		(stroke
@@
 	(wire
 		(pts
-			(xy 242 123) (xy 250 123)
+			(xy 203 124) (xy 211 124)
 		)
 		(stroke
@@
 	(wire
 		(pts
-			(xy 242 129) (xy 250 129)
+			(xy 203 130) (xy 211 130)
 		)
 		(stroke
@@
 	(wire
 		(pts
-			(xy 242 114) (xy 250 114)
-		)
-		(stroke
-			(width 0)
-			(type default)
-		)
-	)
-	(wire
-		(pts
-			(xy 247 141) (xy 250 141)
+			(xy 203 115) (xy 211 115)
+		)
+		(stroke
+			(width 0)
+			(type default)
+		)
+	)
+	(wire
+		(pts
+			(xy 208 142) (xy 211 142)
 		)
 		(stroke
@@
 	(wire
 		(pts
-			(xy 242 138) (xy 250 138)
+			(xy 203 139) (xy 211 139)
 		)
 		(stroke
@@
 	(wire
 		(pts
-			(xy 242 126) (xy 250 126)
+			(xy 203 127) (xy 211 127)
 		)
 		(stroke
@@
 	(hierarchical_label "OUTPUT_0"
 		(shape bidirectional)
-		(at 242 111 180)
+		(at 203 112 180)
 		(effects
 			(font
@@
 	(hierarchical_label "OUTPUT_7"
 		(shape bidirectional)
-		(at 242 132 180)
+		(at 203 133 180)
 		(effects
 			(font
@@
 	(hierarchical_label "OUTPUT_4"
 		(shape bidirectional)
-		(at 242 123 180)
+		(at 203 124 180)
 		(effects
 			(font
@@
 	(hierarchical_label "OUTPUT_1"
 		(shape bidirectional)
-		(at 242 114 180)
+		(at 203 115 180)
 		(effects
 			(font
@@
 	(hierarchical_label "OUTPUT_9"
 		(shape bidirectional)
-		(at 242 138 180)
+		(at 203 139 180)
 		(effects
 			(font
@@
 	(hierarchical_label "OUTPUT_3"
 		(shape bidirectional)
-		(at 242 120 180)
+		(at 203 121 180)
 		(effects
 			(font
@@
 	(hierarchical_label "OUTPUT_2"
 		(shape bidirectional)
-		(at 242 117 180)
+		(at 203 118 180)
 		(effects
 			(font
@@
 	(hierarchical_label "OUTPUT_5"
 		(shape bidirectional)
-		(at 242 126 180)
+		(at 203 127 180)
 		(effects
 			(font
@@
 	(hierarchical_label "OUTPUT_6"
 		(shape bidirectional)
-		(at 242 129 180)
+		(at 203 130 180)
 		(effects
 			(font
@@
 	(hierarchical_label "OUTPUT_8"
 		(shape bidirectional)
-		(at 242 135 180)
+		(at 203 136 180)
 		(effects
 			(font
@@
 	(symbol
 		(lib_id "Generics:J_Connector_1x12")
-		(at 250 108 0)
+		(at 211 109 0)
 		(unit 1)
 		(exclude_from_sim no)
@@
 		(fields_autoplaced yes)
 		(property "Reference" "J8"
-			(at 254 105 0)
+			(at 215 106 0)
 			(do_not_autoplace yes)
 			(effects
@@
 		)
 		(property "Value" "~"
-			(at 219 117 0)
+			(at 180 118 0)
 			(effects
 				(font
@@
 		)
 		(property "Footprint" "Generics:Header_1x12_2.54_TH_labels"
-			(at 219 123 0)
+			(at 180 124 0)
 			(effects
 				(font
@@
 		)
 		(property "Datasheet" ""
-			(at 219 119 0)
+			(at 180 120 0)
 			(effects
 				(font
@@
 		)
 		(property "Description" "Header"
-			(at 254 103 0)
+			(at 215 104 0)
 			(effects
 				(font
@@
 		)
 		(property "Part#" ""
-			(at 250 129 0)
+			(at 211 130 0)
 			(effects
 				(font
@@
 		)
 		(property "Comments" ""
-			(at 250 129 0)
+			(at 211 130 0)
 			(effects
 				(font
@@
 		)
 		(property "PIN_01" "## PIN1"
-			(at 256 108 0)
+			(at 217 109 0)
 			(do_not_autoplace yes)
 			(effects
@@
 		)
 		(property "PIN_02" "## PIN2"
-			(at 256 111 0)
+			(at 217 112 0)
 			(do_not_autoplace yes)
 			(effects
@@
 		)
 		(property "PIN_03" "## PIN3"
-			(at 256 114 0)
+			(at 217 115 0)
 			(do_not_autoplace yes)
 			(effects
@@
 		)
 		(property "PIN_04" "## PIN4"
-			(at 256 117 0)
+			(at 217 118 0)
 			(do_not_autoplace yes)
 			(effects
@@
 		)
 		(property "PIN_05" "## PIN5"
-			(at 256 120 0)
+			(at 217 121 0)
 			(do_not_autoplace yes)
 			(effects
@@
 		)
 		(property "PIN_06" "## PIN6"
-			(at 256 123 0)
+			(at 217 124 0)
 			(do_not_autoplace yes)
 			(effects
@@
 		)
 		(property "PIN_07" "## PIN7"
-			(at 256 126 0)
+			(at 217 127 0)
 			(do_not_autoplace yes)
 			(effects
@@
 		)
 		(property "PIN_08" "## PIN8"
-			(at 256 129 0)
+			(at 217 130 0)
 			(do_not_autoplace yes)
 			(effects
@@
 		)
 		(property "PIN_09" "## PIN9"
-			(at 256 132 0)
+			(at 217 133 0)
 			(do_not_autoplace yes)
 			(effects
@@
 		)
 		(property "PIN_10" "## PIN10"
-			(at 256 135 0)
+			(at 217 136 0)
 			(do_not_autoplace yes)
 			(effects
@@
 		)
 		(property "PIN_11" "## PIN11"
-			(at 256 138 0)
+			(at 217 139 0)
 			(do_not_autoplace yes)
 			(effects
@@
 		)
 		(property "PIN_12" "## PIN12"
-			(at 256 141 0)
+			(at 217 142 0)
 			(do_not_autoplace yes)
 			(effects
@@
 	(symbol
 		(lib_id "Power:VBUS")
-		(at 247 108 0)
+		(at 208 109 0)
 		(unit 1)
 		(exclude_from_sim no)
@@
 		(fields_autoplaced yes)
 		(property "Reference" "#PWR0107"
-			(at 247 121 0)
+			(at 208 122 0)
 			(effects
 				(font
@@
 		)
 		(property "Value" "Vaux_3V3"
-			(at 247 104.19 0)
+			(at 208 105.19 0)
 			(do_not_autoplace yes)
 			(effects
@@
 		)
 		(property "Footprint" ""
-			(at 247 108 0)
+			(at 208 109 0)
 			(effects
 				(font
@@
 		)
 		(property "Datasheet" ""
-			(at 247 108 0)
+			(at 208 109 0)
 			(effects
 				(font
@@
 		)
 		(property "Description" "Power symbol creates a global label with name \"VBUS\""
-			(at 247 119 0)
+			(at 208 120 0)
 			(effects
 				(font
@@
 			)
 		)
-		(property "Footprint" ""
+		(property "Footprint" "Generics:R_0805"
 			(at 206.254 58.984 0)
 			(effects
@@
 			)
 		)
-		(property "Footprint" ""
+		(property "Footprint" "Generics:R_0805"
 			(at 197.254 49.984 0)
 			(effects
@@
 			)
 		)
-		(property "PIN_01" "VCC"
+		(property "PIN_01" "## PIN1"
 			(at 105 55 0)
 			(do_not_autoplace yes)
@@
 			)
 		)
-		(property "PIN_02" "SDA"
+		(property "PIN_02" "## PIN2"
 			(at 105 58 0)
 			(do_not_autoplace yes)
@@
 			)
 		)
-		(property "PIN_03" "SCL"
+		(property "PIN_03" "## PIN3"
 			(at 105 61 0)
 			(do_not_autoplace yes)
@@
 			)
 		)
-		(property "PIN_04" "GND"
+		(property "PIN_04" "## PIN4"
 			(at 105 64 0)
 			(do_not_autoplace yes)
@@
 			)
 		)
-		(property "Footprint" ""
+		(property "Footprint" "Generics:R_0805"
 			(at 197.254 55.984 0)
 			(effects
@@
 			)
 		)
-		(property "Footprint" ""
+		(property "Footprint" "Generics:R_0805"
 			(at 206.254 52.984 0)
 			(effects
@@
 	(symbol
 		(lib_id "Power:GND")
-		(at 247 141 0)
+		(at 208 142 0)
 		(unit 1)
 		(exclude_from_sim no)
@@
 		(fields_autoplaced yes)
 		(property "Reference" "#PWR0108"
-			(at 247 147.35 0)
+			(at 208 148.35 0)
 			(effects
 				(font
@@
 		)
 		(property "Value" "GND"
-			(at 247 144.81 0)
+			(at 208 145.81 0)
 			(effects
 				(font
@@
 		)
 		(property "Footprint" ""
-			(at 247 141 0)
+			(at 208 142 0)
 			(effects
 				(font
@@
 		)
 		(property "Datasheet" ""
-			(at 247 141 0)
+			(at 208 142 0)
 			(effects
 				(font
@@
 		)
 		(property "Description" "Power symbol creates a global label with name \"GND\""
-			(at 249.54 151.668 0)
-			(effects
-				(font
+			(at 210.54 152.668 0)
+			(effects
+				(font

Commit message: DRC / ERC ok
Parts:
- added D14, D15, D16, D17: ~, Generics:D_LED_0603, symbol Generics:D_LED_red
- added R58, R59, R60, R61: 100R, Generics:R_0603, symbol Generics:R
Connections:
- net GND: now also D14.K, D15.K, D16.K, D17.K
- new net: D16.A, R60.1
- new net: D15.A, R59.1
- new net: D17.A, R61.1
- new net: D14.A, R58.1
- new net LED_1: R58.2 (1)
- new net LED_2: R59.2 (1)
- new net LED_3: R60.2 (1)
- new net LED_4: R61.2 (1)
